File: orgonaut66/orgonaut66.kicad_pcb (KiCad board)
At the start: 2 copper layers, 143 parts

Commit message: finsh tracing
Parts:
- D1, D10, D11, D12, D13, D14, D15, D16, D17, D18, D19, D2, D20, D21, D22, D23, D24, D25, D26, D27, D28, D29, D3, D30, D31, D32, D33, D34, D35, D36, D37, D38, D39, D4, D40, D41, D42, D43, D44, D45, D46, D47, D48, D49, D5, D50, D51, D52, D53, D54, D55, D56, D57, D58, D59, D6, D60, D61, D62, D63, D64, D65, D66, D7, D8, D9, J_GND1, J_RGB1, J_VCC1, SW_1: moved to B.Cu
- moved D66 176.5 mm to (317.7, 54.9), turned to 195 degrees
- moved K_RFn1 171.7 mm to (315.6, 65.3), turned to 15 degrees
- moved D59 164.2 mm to (279.6, 6.12), turned to 195 degrees
- moved K_Del1 159.3 mm to (17.8, 13.9), turned to 345 degrees
- moved D3 158.1 mm to (25.2, 6.11), turned to 165 degrees
- moved D62 156.4 mm to (291.8, 42.3), turned to 195 degrees
- moved D60 153.9 mm to (280.3, 25.5), turned to 195 degrees
- moved D65 150.0 mm to (292.1, 61.9), turned to 195 degrees
- moved D9 142.5 mm to (12.7, 61.9), turned to 165 degrees
- moved K_Esc1 141.6 mm to (36.2, 18.8), turned to 345 degrees
- moved D2 140.9 mm to (43.6, 11.0), turned to 165 degrees
- moved D7 139.9 mm to (22.2, 44.8), turned to 165 degrees
- moved D58 138.2 mm to (252.0, 13.5), turned to 195 degrees
- moved D5 137.8 mm to (34.0, 28.2), turned to 165 degrees
- moved D61 130.8 mm to (257.0, 31.9), turned to 195 degrees
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Routing:
- net /row8: track 0.00 -> 491.3 mm, vias 0 -> 1
- net /row7: track 0.00 -> 382.5 mm, vias 0 -> 1
- net /row2: track 0.00 -> 354.3 mm
- net /row4: track 0.00 -> 351.0 mm, vias 0 -> 1
- net /row6: track 0.00 -> 350.3 mm, vias 0 -> 1
- net /col0: track 0.00 -> 315.4 mm
- net /row5: track 0.00 -> 307.7 mm, vias 0 -> 1
- net /col7: track 0.00 -> 289.3 mm
- net /row1: track 0.00 -> 269.0 mm
- net /row3: track 0.00 -> 264.2 mm
- net /col1: track 0.00 -> 255.3 mm
- net /row0: track 0.00 -> 246.2 mm
- net /col6: track 0.00 -> 240.8 mm
- net /col5: track 0.00 -> 195.3 mm
- net /col2: track 0.00 -> 186.1 mm
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- added copper zone on B.Cu, net GND
- added copper zone on F.Cu, net GND
Other:
- board outline added: 361.9 x 150 mm

Commit message: modify tracings & add gerber
Parts:
- moved H5 179.3 mm to (9.53, 28.6)
- moved H6 174.4 mm to (295.3, 28.6)
- moved H2 138.3 mm to (283.4, 90.5)
- moved H1 133.8 mm to (21.4, 90.5)
- moved H4 59.9 mm to (211.9, 123.8)
- moved H3 55.1 mm to (92.9, 123.8)
Routing:
- net /col6: track 240.8 -> 220.8 mm
- net /col5: track 195.3 -> 179.0 mm
- net /col7: track 289.3 -> 287.5 mm

Commit message: update gerber
Other:
- board text added: "The Orgonaut66 in KiCad"
- board text added: "designed by u/lizardsticks"
Changed lines of the file:
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@@
     (area -28.650001 -2.456251 333.450001 147.712501)
     (thickness 1.6)
-    (drawings 9)
+    (drawings 11)
     (tracks 848)
     (zones 0)
@@
     (visible_elements 7FFFF7FF)
     (pcbplotparams
-      (layerselection 0x00030_80000001)
-      (usegerberextensions false)
+      (layerselection 0x010fc_80000001)
+      (usegerberextensions true)
       (excludeedgelayer true)
       (linewidth 0.100000)
@@
       (outputformat 1)
       (mirror false)
-      (drillshape 1)
+      (drillshape 0)
       (scaleselection 1)
-      (outputdirectory ""))
+      (outputdirectory orgonaut66gerber/))
   )
   (net 0 "")
@@
       (net 88 "Net-(U_ProMicro1-Pad24)"))
   )
+  (gr_text "The Orgonaut66 in KiCad" (at 235.74375 121.44375 15) (layer B.Cu)
+    (effects (font (size 1.5 1.5) (thickness 0.3)) (justify mirror))
+  )
+  (gr_text "designed by u/lizardsticks\n" (at 69.05625 121.44375 345) (layer B.Cu)
+    (effects (font (size 1.5 1.5) (thickness 0.3)) (justify mirror))
+  )
   (gr_line (start 21.43125 114.3) (end 154.78125 147.6375) (layer Edge.Cuts) (width 0.15))

Commit message: clean up pcb, update gerber
Parts:
- added H7: Hole, keyboard_parts:HOLE_M2.6, F.Cu at (197.6, 19.1)
- added H8: Hole, keyboard_parts:HOLE_M2.6, F.Cu at (107.2, 19.1)
- moved D22 6.98 mm to (123.8, 52.8)
- moved D16 6.98 mm to (60.0, 70.2)
- moved D10 6.98 mm to (74.7, 15.0)
- moved D12 6.98 mm to (89.4, 33.7)
- moved D13 6.98 mm to (69.8, 33.4)
- moved D15 6.98 mm to (64.9, 51.8)
- moved D2 6.98 mm to (36.7, 9.72)
- moved D20 6.98 mm to (111.5, 24.8)
- moved D21 6.98 mm to (106.6, 43.2)
- moved D23 6.98 mm to (101.7, 61.6)
- moved D4 6.98 mm to (50.2, 33.0)
- moved D18 6.98 mm to (35.4, 88.3)
- moved D26 6.98 mm to (74.7, 88.9)
- moved D32 6.98 mm to (109.0, 108.0)
- moved D3 6.98 mm to (18.3, 4.79)
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Routing:
- net /col7: track 287.5 -> 421.1 mm
- net /col5: track 179.0 -> 299.9 mm
- net /col0: track 315.4 -> 433.6 mm
- net /col2: track 186.1 -> 274.6 mm
- net /col6: track 220.8 -> 295.0 mm
- net /row1: track 269.0 -> 339.8 mm, vias 0 -> 2
- net /col1: track 255.3 -> 323.0 mm
- net /col3: track 126.1 -> 189.5 mm
- net /row0: track 246.2 -> 308.0 mm, vias 0 -> 2
- net /col4: track 118.1 -> 173.7 mm
- net /row3: track 264.2 -> 298.1 mm, vias 0 -> 2
- net /row2: track 354.3 -> 330.9 mm, vias 0 -> 2
- net /row6: track 350.3 -> 372.9 mm, vias 1 -> 2
- net /row4: track 351.0 -> 334.4 mm, vias 1 -> 2
- net /row5: track 307.7 -> 316.8 mm, vias 1 -> 2
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Other:
- board size 361.9 x 150 mm -> 361.9 x 147.6 mm

Commit message: push v2 changes
Routing:
- net /col0: track 433.6 -> 351.4 mm
- net /col7: track 421.1 -> 355.2 mm
- net /col5: track 299.9 -> 239.7 mm
- net /col1: track 323.0 -> 293.7 mm
- net /col4: track 173.7 -> 157.1 mm
- net /col2: track 274.6 -> 258.3 mm
- net /col6: track 295.0 -> 279.9 mm
- net /col3: track 189.5 -> 181.2 mm
