File: orgonaut66/orgonaut66.kicad_pcb (KiCad board)
At the start: 2 copper layers, 361.9 x 147.6 mm, 145 parts

Commit message: push new gerber/ reroute space
Routing:
- net Net-(D33-Pad2): track 15.2 -> 19.1 mm
Changed lines of the file:
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@@
     (thickness 1.6)
     (drawings 13)
-    (tracks 908)
+    (tracks 909)
     (zones 0)
     (modules 145)
@@
     (0 F.Cu signal)
     (31 B.Cu signal)
-    (32 B.Adhes user)
-    (33 F.Adhes user)
+    (32 B.Adhes user hide)
+    (33 F.Adhes user hide)
     (34 B.Paste user)
     (35 F.Paste user)
@@
     (38 B.Mask user)
     (39 F.Mask user)
-    (40 Dwgs.User user)
-    (41 Cmts.User user)
-    (42 Eco1.User user)
-    (43 Eco2.User user)
+    (40 Dwgs.User user hide)
+    (41 Cmts.User user hide)
+    (42 Eco1.User user hide)
+    (43 Eco2.User user hide)
     (44 Edge.Cuts user)
-    (45 Margin user)
-    (46 B.CrtYd user)
-    (47 F.CrtYd user)
-    (48 B.Fab user)
-    (49 F.Fab user)
+    (45 Margin user hide)
+    (46 B.CrtYd user hide)
+    (47 F.CrtYd user hide)
+    (48 B.Fab user hide)
+    (49 F.Fab user hide)
   )
   (setup
@@
     (pcbplotparams
       (layerselection 0x010fc_80000001)
-      (usegerberextensions true)
-      (excludeedgelayer false)
+      (usegerberextensions false)
+      (usegerberattributes true)
+      (excludeedgelayer true)
       (linewidth 0.100000)
       (plotframeref false)
@@
       (psnegative false)
       (psa4output false)
-      (plotreference true)
-      (plotvalue true)
+      (plotreference false)
+      (plotvalue false)
       (plotinvisibletext false)
       (padsonsilk false)
@@
   (segment (start 105.227766 106.962913) (end 105.227766 107.434157) (width 0.25) (layer F.Cu) (net 41) (status 30))
   (segment (start 105.227766 107.434157) (end 110.429216 112.635607) (width 0.25) (layer F.Cu) (net 41) (status 30))
-  (segment (start 136.598689 115.63859) (end 130.87859 115.63859) (width 0.25) (layer F.Cu) (net 42) (status 10))
-  (segment (start 128.905 113.665) (end 122.812716 113.665) (width 0.25) (layer F.Cu) (net 42) (status 20))
-  (segment (start 130.87859 115.63859) (end 128.905 113.665) (width 0.25) (layer F.Cu) (net 42))
+  (segment (start 122.41429 113.266574) (end 122.445426 113.266574) (width 0.25) (layer F.Cu) (net 42))
+  (segment (start 122.445426 113.266574) (end 126.492 109.22) (width 0.25) (layer F.Cu) (net 42))
+  (segment (start 130.180099 109.22) (end 136.598689 115.63859) (width 0.25) (layer F.Cu) (net 42))
+  (segment (start 126.492 109.22) (end 130.180099 109.22) (width 0.25) (layer F.Cu) (net 42))
   (segment (start 122.812716 113.665) (end 122.41429 113.266574) (width 0.25) (layer F.Cu) (net 42) (status 30))
   (segment (start 167.625277 61.312558) (end 167.625277 65.247803) (width 0.25) (layer F.Cu) (net 43) (status 30))
