File: orgonaut66/orgonaut66.kicad_pcb (KiCad board)
At the start: 2 copper layers, 361.9 x 147.6 mm, 145 parts

Commit message: readme
Parts:
- moved H2 94.0 mm to (355.6, 152.2)
- moved H8 94.0 mm to (268.1, 81.2)
- moved H7 94.0 mm to (177.6, 81.2)
- moved K_Down1 94.0 mm to (302.9, 159.6)
- moved K_Period1 94.0 mm to (317.6, 140.9)
- moved K_RFn1 94.0 mm to (387.8, 127.0)
- moved K_RShift1 94.0 mm to (362.5, 133.8)
- moved K_Right1 94.0 mm to (342.1, 159.0)
- moved D37 94.0 mm to (261.3, 151.8)
- moved D41 94.0 mm to (263.7, 87.0)
- moved D53 94.0 mm to (290.7, 114.3)
- moved D54 94.0 mm to (310.4, 114.0)
- moved D59 94.0 mm to (347.8, 69.4)
- moved D60 94.0 mm to (348.1, 89.1)
- moved D63 94.0 mm to (330.0, 113.6)
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Other:
- board size 361.9 x 147.6 mm -> 362 x 147.6 mm

Commit message: update pcb
Parts:
- moved H1 185.7 mm to (292.1, 0.00)
- moved H2 181.8 mm to (301.6, -21.4)
- moved H3 173.9 mm to (152.0, 11.9)
- moved H4 154.1 mm to (125.9, 2.38)
- moved H5 122.7 mm to (142.5, -14.2)
- moved H6 113.2 mm to (330.1, -16.6)
- moved H8 100.4 mm to (315.9, -7.12)
- moved H7 83.6 mm to (175.8, -2.38)
- moved J_GND1 80.8 mm to (208.6, 7.61)
- moved J_RGB1 80.8 mm to (208.7, 1.10)
- moved J_VCC1 80.8 mm to (241.7, 8.09)
- moved SW_1 80.8 mm to (244.3, 2.85)
- moved U_ProMicro1 80.8 mm to (225.2, 14.8)
- moved D3 26.3 mm to (66.3, 80.8), turned to 180 degrees
- moved K_Del1 24.6 mm to (66.4, 89.7), turned to 0 degrees
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Routing:
- net /row8: track 493.8 -> 0.00 mm, vias 2 -> 0
- net /row7: track 382.9 -> 0.00 mm, vias 2 -> 0
- net /row6: track 370.7 -> 0.00 mm, vias 2 -> 0
- net /col7: track 355.2 -> 0.00 mm
- net /col0: track 351.4 -> 0.00 mm
- net /row1: track 336.1 -> 0.00 mm, vias 2 -> 0
- net /row4: track 332.8 -> 0.00 mm, vias 2 -> 0
- net /row2: track 324.8 -> 0.00 mm, vias 2 -> 0
- net /row5: track 302.0 -> 0.00 mm, vias 2 -> 0
- net /col1: track 293.7 -> 0.00 mm
- net /row0: track 292.0 -> 0.00 mm, vias 2 -> 0
- net /row3: track 290.8 -> 0.00 mm, vias 2 -> 0
- net /col6: track 279.7 -> 0.00 mm
- net /col2: track 269.7 -> 0.00 mm
- net /col5: track 239.1 -> 0.00 mm
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- removed copper zone on B.Cu, net GND
- removed copper zone on F.Cu, net GND
Other:
- board outline removed

Commit message: update
Parts:
- U_ProMicro1: moved to B.Cu
- moved H2 276.1 mm to (83.4, 147.7)
- moved H5 257.7 mm to (342.9, 147.7)
- moved H6 204.5 mm to (269.1, 178.6)
- moved H7 184.0 mm to (328.6, 100.0)
- moved H8 177.1 mm to (178.6, 104.8)
- moved H3 166.8 mm to (157.2, 178.7)
- moved H1 113.8 mm to (247.7, 104.8)
- moved H4 101.6 mm to (97.6, 100.0)
- moved J_GND1 81.8 mm to (196.7, 88.6)
- moved J_RGB1 81.8 mm to (196.8, 82.1)
- moved J_VCC1 81.8 mm to (229.8, 89.1)
- moved SW_1 81.8 mm to (232.4, 83.8)
- moved U_ProMicro1 81.8 mm to (213.3, 95.7)
- moved D33 33.3 mm to (178.8, 174.6), turned to 75 degrees
- moved D59 29.3 mm to (337.0, 66.8), turned to 15 degrees
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Connections:
- U_ProMicro1 pad 10: /col1 -> /col6
- U_ProMicro1 pad 11: /col2 -> /col5
- U_ProMicro1 pad 12: /col3 -> /col4
- U_ProMicro1 pad 13: /col4 -> /col3
- U_ProMicro1 pad 14: /col5 -> /col2
- U_ProMicro1 pad 15: /col6 -> /col1
- U_ProMicro1 pad 16: /col7 -> /col0
- U_ProMicro1 pad 9: /col0 -> /col7
Routing:
- net /row8: track 0.00 -> 466.3 mm, vias 0 -> 1
- net /row7: track 0.00 -> 357.8 mm, vias 0 -> 1
- net /row6: track 0.00 -> 327.4 mm, vias 0 -> 1
- net /row4: track 0.00 -> 321.4 mm, vias 0 -> 1
- net /col7: track 0.00 -> 304.0 mm
- net /row2: track 0.00 -> 291.3 mm
- net /col0: track 0.00 -> 289.6 mm
- net /row5: track 0.00 -> 278.7 mm, vias 0 -> 1
- net /row3: track 0.00 -> 250.0 mm, vias 0 -> 1
- net /row1: track 0.00 -> 247.7 mm
- net /col1: track 0.00 -> 242.7 mm
- net /col6: track 0.00 -> 242.5 mm
- net /row0: track 0.00 -> 207.7 mm
- net /col2: track 0.00 -> 201.2 mm
- net /col5: track 0.00 -> 196.0 mm
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- added copper zone on B.Cu, net GND
- added copper zone on F.Cu, net GND
Other:
- board outline added: 350.1 x 138.1 mm

Commit message: update orgonaut v4 for elite c
Parts:
- removed J_GND1, J_RGB1, J_VCC1: Conn_01x01, Connectors:Pin_d0.9mm_L10.0mm_W2.4mm_FlatFork
- removed K_0, K_1, K_2, K_3, K_4, K_5, K_6, K_7, K_8, K_9, K_A1, K_Alt1, K_B1, K_C1, K_Colon1, K_Comma1, K_Ctrl1, K_D1, K_Del1, K_Down1, K_E1, K_Esc1, K_F1, K_G1, K_H1, K_I1, K_J1, K_K1, K_L1, K_LBRC1, K_LFn1, K_Left1, K_Lower1, K_M1, K_N1, K_O1, K_P1, K_Period1, K_PgDn1, K_PgUp1, K_Q1, K_R1, K_RBRC1, K_RFn1, K_Raise1, K_Right1, K_S1, K_Slash1, K_T1, K_U1, K_Up1, K_V1, K_W1, K_Win1, K_X1, K_Y1, K_Z1: KEYSW, keebs:Mx_Alps_100
- removed K_Backspace1, K_Ent1, K_Space1: KEYSW, keebs:Mx_Alps_200
- removed K_Enter1, K_Novelty1: KEYSW, keebs:Mx_Alps_225
- removed K_LShift1: KEYSW, keebs:Mx_Alps_275
- removed K_Pipe1, K_Tab1: KEYSW, keebs:Mx_Alps_150
- removed K_RShift1: KEYSW, keebs:Mx_Alps_175
- removed SW_1: SW_PUSH, Buttons_Switches_SMD:SW_SPST_TL3342
- removed U_ProMicro1: ProMicro, keebs:Pro_Micro
- added D67: WS2812B, Keebio-Parts:RGBW_LED_5mm, F.Cu at (256.5, 61.8)
- added D68: WS2812B, Keebio-Parts:RGBW_LED_5mm, F.Cu at (332.5, 118.8)
- added D69: WS2812B, Keebio-Parts:RGBW_LED_5mm, F.Cu at (142.5, 114.0)
- added D70: WS2812B, Keebio-Parts:RGBW_LED_5mm, F.Cu at (294.5, 57.0)
- added D71: WS2812B, Keebio-Parts:RGBW_LED_5mm, F.Cu at (294.5, 114.0)
- added D72: WS2812B, Keebio-Parts:RGBW_LED_5mm, F.Cu at (104.5, 118.8)
- added D73: WS2812B, Keebio-Parts:RGBW_LED_5mm, F.Cu at (332.5, 61.8)
- added D74: WS2812B, Keebio-Parts:RGBW_LED_5mm, F.Cu at (256.5, 118.8)
- added D75: WS2812B, Keebio-Parts:RGBW_LED_5mm, F.Cu at (92.6, 85.5)
- added D76: WS2812B, Keebio-Parts:RGBW_LED_5mm, F.Cu at (344.4, 85.5)
- added D77: WS2812B, Keebio-Parts:RGBW_LED_5mm, F.Cu at (180.5, 118.8)
- added D78: WS2812B, Keebio-Parts:RGBW_LED_5mm, F.Cu at (104.5, 61.8)
- added D79: WS2812B, Keebio-Parts:RGBW_LED_5mm, F.Cu at (142.5, 57.0)
- added D80: WS2812B, Keebio-Parts:RGBW_LED_5mm, F.Cu at (180.5, 61.8)
- added K1: KEYSW, canadian_footprints:Mx_Alps_100, F.Cu at (66.5, 52.2)
- added K10: KEYSW, canadian_footprints:Mx_Alps_100, F.Cu at (104.5, 128.2)
- added K11: KEYSW, canadian_footprints:Mx_Alps_100, F.Cu at (123.5, 49.9)
- added K12: KEYSW, canadian_footprints:Mx_Alps_100, F.Cu at (123.5, 68.9)
- added K13: KEYSW, canadian_footprints:Mx_Alps_100, F.Cu at (123.5, 87.9)
- added K14: KEYSW, canadian_footprints:Mx_Alps_100, F.Cu at (123.5, 106.9)
- added K15: KEYSW, canadian_footprints:Mx_Alps_100, F.Cu at (123.5, 125.9)
- added K16: KEYSW, canadian_footprints:Mx_Alps_100, F.Cu at (142.5, 47.5)
- added K17: KEYSW, canadian_footprints:Mx_Alps_100, F.Cu at (142.5, 66.5)
- added K18: KEYSW, canadian_footprints:Mx_Alps_100, F.Cu at (142.5, 85.5)
- added K19: KEYSW, canadian_footprints:Mx_Alps_100, F.Cu at (142.5, 104.5)
- added K2: KEYSW, canadian_footprints:Mx_Alps_100, F.Cu at (85.5, 52.2)
- added K20: KEYSW, canadian_footprints:Mx_Alps_100, F.Cu at (142.5, 123.5)
- added K21: KEYSW, canadian_footprints:Mx_Alps_100, F.Cu at (161.5, 49.9)
- added K22: KEYSW, canadian_footprints:Mx_Alps_100, F.Cu at (161.5, 68.9)
- added K23: KEYSW, canadian_footprints:Mx_Alps_100, F.Cu at (161.5, 87.9)
- added K24: KEYSW, canadian_footprints:Mx_Alps_100, F.Cu at (161.5, 106.9)
- added K25: KEYSW, canadian_footprints:Mx_Alps_100, F.Cu at (161.5, 125.9)
- added K26: KEYSW, canadian_footprints:Mx_Alps_100, F.Cu at (180.5, 52.2)
- added K27: KEYSW, canadian_footprints:Mx_Alps_100, F.Cu at (180.5, 71.2)
- added K28: KEYSW, canadian_footprints:Mx_Alps_100, F.Cu at (180.5, 90.2)
- added K29: KEYSW, canadian_footprints:Mx_Alps_100, F.Cu at (180.5, 109.2)
- added K3: KEYSW, canadian_footprints:Mx_Alps_150, F.Cu at (80.8, 71.2)
- added K30: KEYSW, canadian_footprints:Mx_Alps_100, F.Cu at (180.5, 128.2)
- added K31: KEYSW, canadian_footprints:Mx_Alps_100, F.Cu at (199.5, 90.2)
- added K32: KEYSW, canadian_footprints:Mx_Alps_100, F.Cu at (199.5, 109.2)
- added K33: KEYSW, canadian_footprints:Mx_Alps_200-dualside, F.Cu at (199.5, 137.8)
- added K34: KEYSW, canadian_footprints:Mx_Alps_100, F.Cu at (237.5, 90.2)
- added K35: KEYSW, canadian_footprints:Mx_Alps_100, F.Cu at (237.5, 109.2)
- added K36: KEYSW, canadian_footprints:Mx_Alps_200-dualside, F.Cu at (237.5, 137.8)
- added K37: KEYSW, canadian_footprints:Mx_Alps_100, F.Cu at (256.5, 52.2)
- added K38: KEYSW, canadian_footprints:Mx_Alps_100, F.Cu at (256.5, 71.2)
- added K39: KEYSW, canadian_footprints:Mx_Alps_100, F.Cu at (256.5, 90.2)
- added K4: KEYSW, canadian_footprints:Mx_Alps_225, F.Cu at (73.6, 90.2)
- added K40: KEYSW, canadian_footprints:Mx_Alps_100, F.Cu at (256.5, 109.2)
- added K41: KEYSW, canadian_footprints:Mx_Alps_100, F.Cu at (256.5, 128.2)
- added K42: KEYSW, canadian_footprints:Mx_Alps_100, F.Cu at (275.5, 49.9)
- added K43: KEYSW, canadian_footprints:Mx_Alps_100, F.Cu at (275.5, 68.9)
- added K44: KEYSW, canadian_footprints:Mx_Alps_100, F.Cu at (275.5, 87.9)
- added K45: KEYSW, canadian_footprints:Mx_Alps_100, F.Cu at (275.5, 106.9)
- added K46: KEYSW, canadian_footprints:Mx_Alps_100, F.Cu at (275.5, 125.9)
- added K47: KEYSW, canadian_footprints:Mx_Alps_100, F.Cu at (294.5, 47.5)
- added K48: KEYSW, canadian_footprints:Mx_Alps_100, F.Cu at (294.5, 66.5)
- added K49: KEYSW, canadian_footprints:Mx_Alps_100, F.Cu at (294.5, 85.5)
- added K5: KEYSW, canadian_footprints:Mx_Alps_275, F.Cu at (68.9, 109.2)
- added K50: KEYSW, canadian_footprints:Mx_Alps_100, F.Cu at (294.5, 104.5)
- added K51: KEYSW, canadian_footprints:Mx_Alps_100, F.Cu at (294.5, 123.5)
- added K52: KEYSW, canadian_footprints:Mx_Alps_100, F.Cu at (313.5, 49.9)
- added K53: KEYSW, canadian_footprints:Mx_Alps_100, F.Cu at (313.5, 68.9)
- added K54: KEYSW, canadian_footprints:Mx_Alps_100, F.Cu at (313.5, 87.9)
- added K55: KEYSW, canadian_footprints:Mx_Alps_100, F.Cu at (313.5, 106.9)
- added K56: KEYSW, canadian_footprints:Mx_Alps_100, F.Cu at (313.5, 125.9)
- added K57: KEYSW, canadian_footprints:Mx_Alps_100, F.Cu at (332.5, 52.2)
- added K58: KEYSW, canadian_footprints:Mx_Alps_100, F.Cu at (332.5, 71.2)
- added K59: KEYSW, canadian_footprints:Mx_Alps_100, F.Cu at (332.5, 90.2)
- added K6: KEYSW, canadian_footprints:Mx_Alps_100, F.Cu at (104.5, 52.2)
- added K60: KEYSW, canadian_footprints:Mx_Alps_100, F.Cu at (332.5, 109.2)
- added K61: KEYSW, canadian_footprints:Mx_Alps_100, F.Cu at (332.5, 128.2)
- added K62: KEYSW, canadian_footprints:Mx_Alps_200, F.Cu at (361.0, 52.2)
- added K63: KEYSW, canadian_footprints:Mx_Alps_150, F.Cu at (356.2, 71.2)
- added K64: KEYSW, canadian_footprints:Mx_Alps_225, F.Cu at (363.4, 90.2)
- added K65: KEYSW, canadian_footprints:Mx_Alps_175, F.Cu at (358.6, 109.2)
- added K66: KEYSW, canadian_footprints:Mx_Alps_100, F.Cu at (384.8, 109.2)
- added K7: KEYSW, canadian_footprints:Mx_Alps_100, F.Cu at (104.5, 71.2)
- added K8: KEYSW, canadian_footprints:Mx_Alps_100, F.Cu at (104.5, 90.2)
- added K9: KEYSW, canadian_footprints:Mx_Alps_100, F.Cu at (104.5, 109.2)
- added U1: Elite-C, Keebio-Parts:Elite-C-ZigZag, B.Cu at (218.5, 61.8)
- D1, D10, D11, D12, D13, D14, D15, D16, D17, D18, D19, D2, D20, D21, D22, D23, D24, D25, D26, D27, D28, D29, D3, D30, D31, D32, D33, D34, D35, D36, D37, D38, D39, D4, D40, D41, D42, D43, D44, D45, D46, D47, D48, D49, D5, D50, D51, D52, D53, D54, D55, D56, D57, D58, D59, D6, D60, D61, D62, D63, D64, D65, D66, D7, D8, D9: footprint keyboard_parts:D_SOD123_axial -> canadian_footprints:D_SOD123_ThroughHole
- moved H7 236.1 mm to (92.6, 104.5)
- moved H3 201.4 mm to (344.4, 104.5)
- moved H4 171.7 mm to (266.0, 66.5)
- moved H2 119.4 mm to (171.0, 66.5)
- moved H6 108.4 mm to (190.0, 104.5)
- moved D26 106.0 mm to (190.0, 57.0), turned to 90 degrees
- moved D47 94.9 mm to (304.0, 54.6), turned to 90 degrees
- moved H8 94.1 mm to (92.6, 66.5)
- moved D37 93.5 mm to (266.0, 57.0), turned to 90 degrees
- moved D38 92.2 mm to (266.0, 76.0), turned to 90 degrees
- moved D57 91.8 mm to (342.0, 57.0), turned to 90 degrees
- moved D48 90.0 mm to (304.0, 73.6), turned to 90 degrees
- moved D27 89.7 mm to (190.0, 76.0), turned to 90 degrees
- moved D17 82.4 mm to (152.0, 73.6), turned to 90 degrees
- moved D39 81.8 mm to (266.0, 95.0), turned to 90 degrees
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Connections:
- D10 pad 1: /row0 -> /row4
- D11 pad 1: /row1 -> /row0
- D12 pad 1: /row2 -> /row1
- D13 pad 1: /row3 -> /row2
- D14 pad 1: /row4 -> /row3
- D15 pad 1: /row5 -> /row4
- D16 pad 1: /row6 -> /row0
- D17 pad 1: /row7 -> /row1
- D18 pad 1: /row8 -> /row2
- D19 pad 1: /row0 -> /row3
- D20 pad 1: /row1 -> /row4
- D21 pad 1: /row2 -> /row0
- D22 pad 1: /row3 -> /row1
- D23 pad 1: /row4 -> /row2
- D24 pad 1: /row5 -> /row3
- D25 pad 1: /row6 -> /row4
- D26 pad 1: /row7 -> /row0
- D27 pad 1: /row8 -> /row1
- D28 pad 1: /row3 -> /row2
- D29 pad 1: /row4 -> /row3
- D30 pad 1: /row5 -> /row4
- D31 pad 1: /row6 -> /row2
- D32 pad 1: /row7 -> /row3
- D33 pad 1: /row8 -> /row4
- D34 pad 1: /row3 -> /row2
- D35 pad 1: /row4 -> /row3
- D36 pad 1: /row5 -> /row4
- D37 pad 1: /row6 -> /row0
- D38 pad 1: /row7 -> /row1
- D39 pad 1: /row8 -> /row2
- D40 pad 1: /row0 -> /row3
- D41 pad 1: /row1 -> /row4
- D42 pad 1: /row2 -> /row0
- D43 pad 1: /row3 -> /row1
- D44 pad 1: /row4 -> /row2
- D45 pad 1: /row5 -> /row3
- D46 pad 1: /row6 -> /row4
- D47 pad 1: /row7 -> /row0
- D48 pad 1: /row8 -> /row1
- D49 pad 1: /row0 -> /row2
- D50 pad 1: /row1 -> /row3
- D51 pad 1: /row2 -> /row4
- D52 pad 1: /row3 -> /row0
- D53 pad 1: /row4 -> /row1
- D54 pad 1: /row5 -> /row2
- D55 pad 1: /row6 -> /row3
- D56 pad 1: /row7 -> /row4
- D57 pad 1: /row8 -> /row0
- D58 pad 1: /row0 -> /row1
- D59 pad 1: /row1 -> /row2
- D6 pad 1: /row5 -> /row0
- D60 pad 1: /row2 -> /row3
- D61 pad 1: /row3 -> /row4
- D62 pad 1: /row4 -> /row0
- D63 pad 1: /row5 -> /row1
- D64 pad 1: /row6 -> /row2
- D65 pad 1: /row7 -> /row3
- D66 pad 1: /row8 -> /row4
- D7 pad 1: /row6 -> /row1
- D8 pad 1: /row7 -> /row2
- D9 pad 1: /row8 -> /row3
Routing:
- net VCC: track 25.0 -> 522.3 mm, vias 0 -> 26
- net /row8: track 466.3 -> 0.00 mm, vias 1 -> 0
- net /row7: track 357.8 -> 0.00 mm, vias 1 -> 0
- net /row6: track 327.4 -> 0.00 mm, vias 1 -> 0
- net /row5: track 278.7 -> 0.00 mm, vias 1 -> 0
- net /col7: track 304.0 -> 50.0 mm
- net /col0: track 289.6 -> 90.0 mm
- net /col6: track 242.5 -> 48.1 mm
- net /col1: track 242.7 -> 76.0 mm
- net /col2: track 201.2 -> 76.0 mm
- net /col5: track 196.0 -> 76.0 mm
- net /col4: track 127.4 -> 19.0 mm
- net /cold: track 0.00 -> 88.6 mm
- net /colc: track 0.00 -> 76.0 mm
- net /colb: track 0.00 -> 76.0 mm
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- removed copper zone on B.Cu, net GND
- removed copper zone on F.Cu, net GND
Other:
- board size 350.1 x 138.1 mm -> 356.2 x 123.5 mm
- board text removed: "The Orgonaut66 in KiCad"
- board text removed: "designed by u/lizardsticks"
