File: orgonaut66/orgonaut66.sch (KiCad schematic (older format))
At the start: 143 parts

Commit message: clean up pcb, update gerber
Parts:
- added H7, H8: Hole, keyboard_parts:HOLE_M2.6, symbol Hole
Other:
- moved on the sheet: H1, H2, H3, H4, H5, H6
Changed lines of the file:
@@
 LIBS:contrib
 LIBS:valves
-LIBS:ergo60tilt-cache
+LIBS:orgonaut66-cache
 EELAYER 25 0
 EELAYER END
@@
 L Hole H3
 U 1 1 5B91704E
-P 6050 6600
-F 0 "H3" H 6050 6550 60  0000 C CNN
-F 1 "Hole" H 6050 6650 60  0000 C CNN
-F 2 "keyboard_parts:HOLE_M2.6" H 6050 6600 60  0001 C CNN
-F 3 "" H 6050 6600 60  0001 C CNN
-	1    6050 6600
+P 5600 6600
+F 0 "H3" H 5600 6550 60  0000 C CNN
+F 1 "Hole" H 5600 6650 60  0000 C CNN
+F 2 "keyboard_parts:HOLE_M2.6" H 5600 6600 60  0001 C CNN
+F 3 "" H 5600 6600 60  0001 C CNN
+	1    5600 6600
 	1    0    0    -1
 $EndComp
@@
 L Hole H4
 U 1 1 5B91704F
-P 6050 7100
-F 0 "H4" H 6050 7050 60  0000 C CNN
-F 1 "Hole" H 6050 7150 60  0000 C CNN
-F 2 "keyboard_parts:HOLE_M2.6" H 6050 7100 60  0001 C CNN
-F 3 "" H 6050 7100 60  0001 C CNN
-	1    6050 7100
+P 5600 7100
+F 0 "H4" H 5600 7050 60  0000 C CNN
+F 1 "Hole" H 5600 7150 60  0000 C CNN
+F 2 "keyboard_parts:HOLE_M2.6" H 5600 7100 60  0001 C CNN
+F 3 "" H 5600 7100 60  0001 C CNN
+	1    5600 7100
 	1    0    0    -1
 $EndComp
@@
 L Hole H1
 U 1 1 5B917050
-P 5500 6600
-F 0 "H1" H 5500 6550 60  0000 C CNN
-F 1 "Hole" H 5500 6650 60  0000 C CNN
-F 2 "keyboard_parts:HOLE_M2.6" H 5500 6600 60  0001 C CNN
-F 3 "" H 5500 6600 60  0001 C CNN
-	1    5500 6600
+P 5050 6600
+F 0 "H1" H 5050 6550 60  0000 C CNN
+F 1 "Hole" H 5050 6650 60  0000 C CNN
+F 2 "keyboard_parts:HOLE_M2.6" H 5050 6600 60  0001 C CNN
+F 3 "" H 5050 6600 60  0001 C CNN
+	1    5050 6600
 	1    0    0    -1
 $EndComp
@@
 L Hole H2
 U 1 1 5B917051
-P 5500 7100
-F 0 "H2" H 5500 7050 60  0000 C CNN
-F 1 "Hole" H 5500 7150 60  0000 C CNN
-F 2 "keyboard_parts:HOLE_M2.6" H 5500 7100 60  0001 C CNN
-F 3 "" H 5500 7100 60  0001 C CNN
-	1    5500 7100
+P 5050 7100
+F 0 "H2" H 5050 7050 60  0000 C CNN
+F 1 "Hole" H 5050 7150 60  0000 C CNN
+F 2 "keyboard_parts:HOLE_M2.6" H 5050 7100 60  0001 C CNN
+F 3 "" H 5050 7100 60  0001 C CNN
+	1    5050 7100
 	1    0    0    -1
 $EndComp
@@
 L Hole H5
 U 1 1 5B917052
-P 6600 6600
-F 0 "H5" H 6600 6550 60  0000 C CNN
-F 1 "Hole" H 6600 6650 60  0000 C CNN
-F 2 "keyboard_parts:HOLE_M2.6" H 6600 6600 60  0001 C CNN
-F 3 "" H 6600 6600 60  0001 C CNN
-	1    6600 6600
+P 6150 6600
+F 0 "H5" H 6150 6550 60  0000 C CNN
+F 1 "Hole" H 6150 6650 60  0000 C CNN
+F 2 "keyboard_parts:HOLE_M2.6" H 6150 6600 60  0001 C CNN
+F 3 "" H 6150 6600 60  0001 C CNN
+	1    6150 6600
 	1    0    0    -1
 $EndComp
@@
 L Hole H6
 U 1 1 5B917053
-P 6600 7100
-F 0 "H6" H 6600 7050 60  0000 C CNN
-F 1 "Hole" H 6600 7150 60  0000 C CNN
-F 2 "keyboard_parts:HOLE_M2.6" H 6600 7100 60  0001 C CNN
-F 3 "" H 6600 7100 60  0001 C CNN
-	1    6600 7100
+P 6150 7100
+F 0 "H6" H 6150 7050 60  0000 C CNN
+F 1 "Hole" H 6150 7150 60  0000 C CNN
+F 2 "keyboard_parts:HOLE_M2.6" H 6150 7100 60  0001 C CNN
+F 3 "" H 6150 7100 60  0001 C CNN
+	1    6150 7100
 	1    0    0    -1
 $EndComp
@@
 Wire Wire Line
 	3500 7300 3500 7450
+$Comp
+L Hole H7
+U 1 1 5B92D62B
+P 6650 6600
+F 0 "H7" H 6650 6550 60  0000 C CNN
+F 1 "Hole" H 6650 6650 60  0000 C CNN
+F 2 "keyboard_parts:HOLE_M2.6" H 6650 6600 60  0001 C CNN
+F 3 "" H 6650 6600 60  0001 C CNN
+	1    6650 6600
+	1    0    0    -1
+$EndComp
+$Comp
+L Hole H8
+U 1 1 5B92D631
+P 6650 7100
+F 0 "H8" H 6650 7050 60  0000 C CNN
+F 1 "Hole" H 6650 7150 60  0000 C CNN
+F 2 "keyboard_parts:HOLE_M2.6" H 6650 7100 60  0001 C CNN
+F 3 "" H 6650 7100 60  0001 C CNN
+	1    6650 7100
+	1    0    0    -1
+$EndComp
 $EndSCHEMATC

Commit message: update
Connections:
- net col0: now also U_ProMicro1.16 (15/PB1); no longer U_ProMicro1.9 (6/PD7)
- net col1: now also U_ProMicro1.15 (14/PB3); no longer U_ProMicro1.10 (7/PE6)
- net col2: now also U_ProMicro1.14 (16/PB2); no longer U_ProMicro1.11 (8/PB4)
- net col3: now also U_ProMicro1.13 (10/PB6); no longer U_ProMicro1.12 (9/PB5)
- net col4: now also U_ProMicro1.12 (9/PB5); no longer U_ProMicro1.13 (10/PB6)
- net col5: now also U_ProMicro1.11 (8/PB4); no longer U_ProMicro1.14 (16/PB2)
- net col6: now also U_ProMicro1.10 (7/PE6); no longer U_ProMicro1.15 (14/PB3)
- net col7: now also U_ProMicro1.9 (6/PD7); no longer U_ProMicro1.16 (15/PB1)

Commit message: update orgonaut v4 for elite c
Parts:
- removed D1, D10, D11, D12, D13, D14, D15, D16, D17, D18, D19, D2, D20, D21, D22, D23, D24, D25, D26, D27, D28, D29, D3, D30, D31, D32, D33, D34, D35, D36, D37, D38, D39, D4, D40, D41, D42, D43, D44, D45, D46, D47, D48, D49, D5, D50, D51, D52, D53, D54, D55, D56, D57, D58, D59, D6, D60, D61, D62, D63, D64, D65, D66, D7, D8, D9: D, keyboard_parts:D_SOD123_axial, symbol D
- removed H1, H2, H3, H4, H5, H6, H7, H8: Hole, keyboard_parts:HOLE_M2.6, symbol Hole
- removed J_GND1, J_RGB1, J_VCC1: Conn_01x01, Connectors:Pin_d0.9mm_L10.0mm_W2.4mm_FlatFork, symbol Conn_01x01
- removed K_0, K_1, K_2, K_3, K_4, K_5, K_6, K_7, K_8, K_9, K_A1, K_Alt1, K_B1, K_C1, K_Colon1, K_Comma1, K_Ctrl1, K_D1, K_Del1, K_Down1, K_E1, K_Esc1, K_F1, K_G1, K_H1, K_I1, K_J1, K_K1, K_L1, K_LBRC1, K_LFn1, K_Left1, K_Lower1, K_M1, K_N1, K_O1, K_P1, K_Period1, K_PgDn1, K_PgUp1, K_Q1, K_R1, K_RBRC1, K_RFn1, K_Raise1, K_Right1, K_S1, K_Slash1, K_T1, K_U1, K_Up1, K_V1, K_W1, K_Win1, K_X1, K_Y1, K_Z1: KEYSW, keebs:Mx_Alps_100, symbol KEYSW
- removed K_Backspace1, K_Ent1, K_Space1: KEYSW, keebs:Mx_Alps_200, symbol KEYSW
- removed K_Enter1, K_Novelty1: KEYSW, keebs:Mx_Alps_225, symbol KEYSW
- removed K_LShift1: KEYSW, keebs:Mx_Alps_275, symbol KEYSW
- removed K_Pipe1, K_Tab1: KEYSW, keebs:Mx_Alps_150, symbol KEYSW
- removed K_RShift1: KEYSW, keebs:Mx_Alps_175, symbol KEYSW
- removed SW_1: SW_PUSH, Buttons_Switches_SMD:SW_SPST_TL3342, symbol SW_PUSH
- removed U_ProMicro1: ProMicro, keebs:Pro_Micro, symbol ProMicro
- added D1, D10, D11, D12, D13, D14, D15, D16, D17, D18, D19, D2, D20, D21, D22, D23, D24, D25, D26, D27, D28, D29, D3, D30, D31, D32, D33, D34, D35, D36, D37, D38, D39, D4, D40, D41, D42, D43, D44, D45, D46, D47, D48, D49, D5, D50, D51, D52, D53, D54, D55, D56, D57, D58, D59, D6, D60, D61, D62, D63, D64, D65, D66, D7, D8, D9: D, canadian_footprints:D_SOD123_ThroughHole, symbol Device:D
- added D67, D68, D69, D70, D71, D72, D73, D74, D75, D76, D77, D78, D79, D80: WS2812B, Keebio-Parts:RGBW_LED_5mm, symbol LED:WS2812B
- added H1, H2, H3, H4, H5, H6, H7, H8: Hole, keyboard_parts:Poker_oval_hole, symbol keebio:Hole
- added K1, K10, K11, K12, K13, K14, K15, K16, K17, K18, K19, K2, K20, K21, K22, K23, K24, K25, K26, K27, K28, K29, K30, K31, K32, K34, K35, K37, K38, K39, K40, K41, K42, K43, K44, K45, K46, K47, K48, K49, K50, K51, K52, K53, K54, K55, K56, K57, K58, K59, K6, K60, K61, K66, K7, K8, K9: KEYSW, canadian_footprints:Mx_Alps_100, symbol keyboard_parts:KEYSW
- added K3, K63: KEYSW, canadian_footprints:Mx_Alps_150, symbol keyboard_parts:KEYSW
- added K33, K36: KEYSW, canadian_footprints:Mx_Alps_200-dualside, symbol keyboard_parts:KEYSW
- added K4, K64: KEYSW, canadian_footprints:Mx_Alps_225, symbol keyboard_parts:KEYSW
- added K5: KEYSW, canadian_footprints:Mx_Alps_275, symbol keyboard_parts:KEYSW
- added K62: KEYSW, canadian_footprints:Mx_Alps_200, symbol keyboard_parts:KEYSW
- added K65: KEYSW, canadian_footprints:Mx_Alps_175, symbol keyboard_parts:KEYSW
- added U1: Elite-C, Keebio-Parts:Elite-C-ZigZag, symbol keebio:Elite-C
Connections:
- net GND: now also D67.3 (VSS), D68.3 (VSS), D69.3 (VSS), D70.3 (VSS), D71.3 (VSS), D72.3 (VSS), D73.3 (VSS), D74.3 (VSS), D75.3 (VSS), D76.3 (VSS), D77.3 (VSS), D78.3 (VSS), D79.3 (VSS), D80.3 (VSS), U1.23 (GND), U1.3 (GND), U1.4 (GND)
- net RGB: now also D67.4 (DIN), U1.1 (TX0/PD3)
- net VCC: now also D67.1 (VDD), D68.1 (VDD), D69.1 (VDD), D70.1 (VDD), D71.1 (VDD), D72.1 (VDD), D73.1 (VDD), D74.1 (VDD), D75.1 (VDD), D76.1 (VDD), D77.1 (VDD), D78.1 (VDD), D79.1 (VDD), D80.1 (VDD), U1.21 (VCC)
- net col0: now also K1.1, K2.1, K3.1, K4.1, K5.1, U1.19 (A2/PF5)
- net col1: now also K10.1, K6.1, K7.1, K8.1, K9.1, U1.18 (A1/PF6)
- net col2: now also K11.1, K12.1, K13.1, K14.1, K15.1, U1.17 (A0/PF7)
- net col3: now also K16.1, K17.1, K18.1, K19.1, K20.1, U1.16 (15/PB1)
- net col4: now also K21.1, K22.1, K23.1, K24.1, K25.1, U1.15 (14/PB3)
- net col5: now also K26.1, K27.1, K28.1, K29.1, K30.1, U1.14 (16/PB2)
- net col6: now also K31.1, K32.1, K33.1, U1.13 (10/PB6)
- net col7: now also K34.1, K35.1, K36.1, U1.12 (9/PB5)
- net row0: now also D1.1 (K), D11.1 (K), D16.1 (K), D21.1 (K), D26.1 (K), D37.1 (K), D42.1 (K), D47.1 (K), D52.1 (K), D57.1 (K), D6.1 (K), D62.1 (K), U1.25 (B7)
- net row1: now also D12.1 (K), D17.1 (K), D2.1 (K), D22.1 (K), D27.1 (K), D38.1 (K), D43.1 (K), D48.1 (K), D53.1 (K), D58.1 (K), D63.1 (K), D7.1 (K), U1.26 (D5)
- net row2: now also D13.1 (K), D18.1 (K), D23.1 (K), D28.1 (K), D3.1 (K), D31.1 (K), D34.1 (K), D39.1 (K), D44.1 (K), D49.1 (K), D54.1 (K), D59.1 (K), D64.1 (K), D8.1 (K), U1.27 (C7)
- net row3: now also D14.1 (K), D19.1 (K), D24.1 (K), D29.1 (K), D32.1 (K), D35.1 (K), D4.1 (K), D40.1 (K), D45.1 (K), D50.1 (K), D55.1 (K), D60.1 (K), D65.1 (K), D9.1 (K), U1.28 (F1)
- net row4: now also D10.1 (K), D15.1 (K), D20.1 (K), D25.1 (K), D30.1 (K), D33.1 (K), D36.1 (K), D41.1 (K), D46.1 (K), D5.1 (K), D51.1 (K), D56.1 (K), D61.1 (K), D66.1 (K), U1.29 (F0)
- new net: D1.2 (A), K1.2
- new net: D2.2 (A), K2.2
- new net: D3.2 (A), K3.2
- new net: D4.2 (A), K4.2
- new net: D5.2 (A), K5.2
- new net: D6.2 (A), K6.2
- new net: D7.2 (A), K7.2
- new net: D8.2 (A), K8.2
- new net: D9.2 (A), K9.2
- new net: D10.2 (A), K10.2
- new net: D11.2 (A), K11.2
- new net: D12.2 (A), K12.2
- new net: D13.2 (A), K13.2
- new net: D14.2 (A), K14.2
- new net: D15.2 (A), K15.2
- new net: D16.2 (A), K16.2
- new net: D17.2 (A), K17.2
- new net: D18.2 (A), K18.2
- new net: D19.2 (A), K19.2
- new net: D20.2 (A), K20.2
- new net: D21.2 (A), K21.2
- new net: D22.2 (A), K22.2
- new net: D23.2 (A), K23.2
- new net: D24.2 (A), K24.2
- new net: D25.2 (A), K25.2
- new net: D26.2 (A), K26.2
- new net: D27.2 (A), K27.2
- new net: D28.2 (A), K28.2
- new net: D29.2 (A), K29.2
- new net: D30.2 (A), K30.2
- new net: D31.2 (A), K31.2
- new net: D32.2 (A), K32.2
- new net: D33.2 (A), K33.2
- new net: D34.2 (A), K34.2
- new net: D35.2 (A), K35.2
- new net: D36.2 (A), K36.2
- new net: D37.2 (A), K37.2
- new net: D38.2 (A), K38.2
- new net: D39.2 (A), K39.2
- new net: D40.2 (A), K40.2
- new net: D41.2 (A), K41.2
- new net: D42.2 (A), K42.2
- new net: D43.2 (A), K43.2
- new net: D44.2 (A), K44.2
- new net: D45.2 (A), K45.2
- new net: D46.2 (A), K46.2
- new net: D47.2 (A), K47.2
- new net: D48.2 (A), K48.2
- new net: D49.2 (A), K49.2
- new net: D50.2 (A), K50.2
- new net: D51.2 (A), K51.2
- new net: D52.2 (A), K52.2
- new net: D53.2 (A), K53.2
- new net: D54.2 (A), K54.2
- new net: D55.2 (A), K55.2
- new net: D56.2 (A), K56.2
- new net: D57.2 (A), K57.2
- new net: D58.2 (A), K58.2
- new net: D59.2 (A), K59.2
- new net: D60.2 (A), K60.2
- new net: D61.2 (A), K61.2
- new net: D62.2 (A), K62.2
- new net: D63.2 (A), K63.2
- new net: D64.2 (A), K64.2
- new net: D65.2 (A), K65.2
- new net: D66.2 (A), K66.2
- new net: D79.2 (DOUT), D80.4 (DIN)
- new net: D78.2 (DOUT), D79.4 (DIN)
- new net: D67.2 (DOUT), D70.4 (DIN)
- new net: D70.2 (DOUT), D73.4 (DIN)
- new net: D73.2 (DOUT), D76.4 (DIN)
- new net: D68.4 (DIN), D76.2 (DOUT)
- new net: D68.2 (DOUT), D71.4 (DIN)
- new net: D71.2 (DOUT), D74.4 (DIN)
- new net: D74.2 (DOUT), D77.4 (DIN)
- new net: D69.4 (DIN), D77.2 (DOUT)
- new net: D69.2 (DOUT), D72.4 (DIN)
- new net: D72.2 (DOUT), D75.4 (DIN)
- new net: D75.2 (DOUT), D78.4 (DIN)
- new net col8: K37.1, K38.1, K39.1, K40.1, K41.1, U1.11 (8/PB4)
- new net col9: K42.1, K43.1, K44.1, K45.1, K46.1, U1.10 (7/PE6)
- new net cola: K47.1, K48.1, K49.1, K50.1, K51.1, U1.9 (6/PD7)
- new net colb: K52.1, K53.1, K54.1, K55.1, K56.1, U1.8 (5/PC6)
- new net colc: K57.1, K58.1, K59.1, K60.1, K61.1, U1.7 (4/PD4)
- new net cold: K62.1, K63.1, K64.1, K65.1, K66.1, U1.6 (3/PD0)
- no-connect marks 1 -> 6
Other:
- note removed: "The OrgoNaut 66 by u/lizardsticks\n\n"
